Commit message: update doc for robots + add grippers

File: pyrobolearn/robots/urdfs/allegrohand/allegro_right_hand.urdf (robot description, URDF)
Before this commit: robot allegro_hand_right, 22 links, 21 joints
Links:
- removed link box_link
Joints:
- removed joint box_to_base

File: pyrobolearn/robots/urdfs/shadowhand/left_hand.urdf (robot description, URDF)
Before this commit: robot shadowhand_motor, 33 links, 32 joints
Links:
- removed link world
Joints:
- removed joint lh_world_joint

File: pyrobolearn/robots/urdfs/shadowhand/right_hand.urdf (robot description, URDF)
Before this commit: robot shadowhand_motor, 33 links, 32 joints
Links:
- removed link world
Joints:
- removed joint rh_world_joint

File: pyrobolearn/robots/urdfs/softhand/left_hand.urdf (robot description, URDF)
Before this commit: robot soft_hand, 39 links, 38 joints
Links:
- link left_hand_kuka_coupler_bottom: mass 0 -> 1.e-6

File: pyrobolearn/robots/urdfs/softhand/right_hand.urdf (robot description, URDF)
Before this commit: robot soft_hand, 39 links, 38 joints
Links:
- link right_hand_kuka_coupler_bottom: mass 0 -> 1.e-6
